File: 5116-05/LM5116-05.kicad_sch (KiCad schematic)
At the start: 44 parts, among them J1 Input, J3 40HAT, J6 CONN_02X02, J9 CONN_01X02, Q1 DMG2305UX, Q2 DMMT5401, Q3 CSD19534Q5A, Q4 IPB027N10N3_G, U1 LM5116MHX_NOPB, U2 CAT24C32

Commit message: routed V05
Connections:
- net GND: now also C1.1
- net Vin: now reaches Cin1.1, Cinx1.1, J1.2 (Pin_2), Q3.5 (D), Renable1.1, Ruv2.1, U1.1 (VIN)
- net q4_pad3: now reaches Q4.3, Rsense1.1, U1.12 (CS)
- net lo: now reaches Q4.1, U1.15 (LO)
- net ho: now reaches Q3.4 (G), U1.19 (HO)
- no-connect marks 27 -> 26
