File: 5116-05/LM5116-05.kicad_pcb (KiCad board)
At the start: 2 copper layers, 65 x 56 mm, 49 parts, among them J1 Input, J3 40HAT, J6 CONN_02X02, J9 CONN_01X02, Q1 DMG2305UX, Q2 DMMT5401, Q3 CSD19534Q5A, Q4 IPB027N10N3_G, U1 LM5116MHX_NOPB, U2 CAT24C32

Commit message: routed V05
Parts:
- added TP_5V: test_point, Connector_Pin:test_point, F.Cu at (110.5, 82.3)
- moved L1 98.3 mm to (87.6, 83.8), turned to 90 degrees
- moved Cout1 95.9 mm to (100.6, 78.5), turned to 90 degrees
- moved Q3 80.1 mm to (88.1, 94.5), turned to -90 degrees
- moved Rfbt1 77.8 mm to (114.4, 87.1), turned to 0 degrees
- moved Q4 77.2 mm to (96.8, 90.9), turned to 90 degrees
- moved Rfbb1 77.1 mm to (118.6, 87.9), turned to 0 degrees
- moved Ccomp1 72.6 mm to (117.0, 89.9), turned to 180 degrees
- moved Cvcc1 71.4 mm to (103.4, 91.8), turned to 90 degrees
- moved Rcomp1 70.7 mm to (115.2, 90.7), turned to 90 degrees
- moved Ccomp2 69.1 mm to (116.9, 91.7), turned to 180 degrees
- moved TP_Q 64.8 mm to (103.4, 83.8)
- moved Css1 64.6 mm to (117.1, 94.0), turned to 0 degrees
- moved D1 64.6 mm to (103.6, 95.1), turned to 90 degrees
- moved U1 63.4 mm to (109.4, 94.5), turned to 180 degrees
- moved Cin1 61.1 mm to (92.5, 102.4), turned to 0 degrees
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Connections:
- net Net-(Cin1-Pad1) renamed Vin
- net Net-(Q3-Pad4) renamed ho
- net Net-(Q4-Pad1) renamed lo
- C1 pad 1: unconnected-(C1-Pad1) -> GND
- TP_Q pad 1: Net-(Cboot1-Pad2) -> cont
- TP_SYNC pad 1: Net-(C1-Pad1) -> Net-(C1-Pad2)
Routing:
- net Vin: track 0.00 -> 30.9 mm
- net ho: track 1.65 -> 29.2 mm
- net Net-(C1-Pad2): track 0.00 -> 18.6 mm
- net GND: track 3.81 -> 22.2 mm, vias 0 -> 16
- net Net-(Renable1-Pad2): track 0.00 -> 17.0 mm, vias 0 -> 2
- net /P5V: track 10.3 -> 26.2 mm
- net cont: track 1.80 -> 15.3 mm, vias 1 -> 17
- net lo: track 0.00 -> 13.4 mm, vias 0 -> 2
- net Net-(Ccomp1-Pad1): track 0.00 -> 12.8 mm
- net Net-(Ruv1-Pad1): track 0.00 -> 8.27 mm
- net q4_pad3: track 1.53 -> 9.68 mm, vias 1 -> 3
- net Net-(Cvcc1-Pad1): track 0.00 -> 5.06 mm
- net Net-(Ccomp2-Pad2): track 0.00 -> 4.80 mm
- net Net-(Cramp1-Pad1): track 0.00 -> 4.32 mm
- net Net-(Cboot1-Pad1): track 0.00 -> 4.21 mm
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- added copper zone on B.Cu, net GND
- added copper zone on F.Cu, net GND
- added copper zone on F.Cu, net Vin
- added copper zone on B.Cu, net cont
- added copper zone on F.Cu, net cont
- added copper zone on B.Cu, net ho
- added copper zone on B.Cu, net lo
- added copper zone on F.Cu, net lo

Commit message: Added Gerbers
Parts:
- moved Cinx1 0.51 mm to (111.5, 99.3)
Other:
- rule pad_to_mask_clearance: 0.1 -> 0
- board text removed: "order q2 & lm5116"
Changed lines of the file:
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@@
       (dielectric_constraints no)
     )
-    (pad_to_mask_clearance 0.1)
+    (pad_to_mask_clearance 0)
     (pcbplotparams
-      (layerselection 0x00210fc_ffffffff)
+      (layerselection 0x00010fc_ffffffff)
       (disableapertmacros false)
-      (usegerberextensions false)
+      (usegerberextensions true)
       (usegerberattributes false)
       (usegerberadvancedattributes false)
@@
       (plotinvisibletext false)
       (sketchpadsonfab false)
-      (subtractmaskfromsilk false)
+      (subtractmaskfromsilk true)
       (outputformat 1)
       (mirror false)
       (drillshape 0)
       (scaleselection 1)
-      (outputdirectory "prod-03")
+      (outputdirectory "05_gerber/")
     )
   )
@@
     (property "Sheetname" "")
     (attr smd)
-    (fp_text reference "R7" (at 0 -1.65) (layer "F.SilkS")
+    (fp_text reference "R7" (at 2.55 -0.046) (layer "F.SilkS")
       (effects (font (size 1 1) (thickness 0.15)))
     )
@@
     (property "Sheetname" "")
     (attr through_hole)
-    (fp_text reference "J6" (at 1.27 -2.33 180) (layer "F.SilkS")
+    (fp_text reference "J6" (at -2.54 3.302 180) (layer "F.SilkS")
       (effects (font (size 1 1) (thickness 0.15)))
     )
@@
     (fp_line (start -1.6 1.25) (end -1.6 -1.25) (layer "F.Fab") (width 0.1))
     (fp_line (start 1.6 1.25) (end -1.6 1.25) (layer "F.Fab") (width 0.1))
-    (pad "1" smd roundrect (at -1.475 0) (size 1.15 2.7) (layers "F.Cu" "F.Paste" "F.Mask") (roundrect_rratio 0.217391)
+    (pad "1" smd roundrect (at -1.475 0) (size 1.15 2.7) (layers "F.Cu" "F.Paste" "F.Mask") (roundrect_rratio 0.2173913043)
       (net 51 "Vin") (pintype "passive"))
-    (pad "2" smd roundrect (at 1.475 0) (size 1.15 2.7) (layers "F.Cu" "F.Paste" "F.Mask") (roundrect_rratio 0.217391)
+    (pad "2" smd roundrect (at 1.475 0) (size 1.15 2.7) (layers "F.Cu" "F.Paste" "F.Mask") (roundrect_rratio 0.2173913043)
       (net 1 "GND") (pintype "passive"))
     (model "${KICAD6_3DMODEL_DIR}/Capacitor_SMD.3dshapes/C_1210_3225Metric.wrl"
@@
     (property "Sheetname" "")
     (attr smd)
-    (fp_text reference "D2" (at 0 -1.65) (layer "F.SilkS")
+    (fp_text reference "D2" (at -0.254 1.778) (layer "F.SilkS")
       (effects (font (size 1 1) (thickness 0.15)))
     )
@@
     (property "Sheetname" "")
     (attr smd)
-    (fp_text reference "R1" (at 0 -1.65) (layer "F.SilkS")
+    (fp_text reference "R1" (at 0.254 1.778) (layer "F.SilkS")
       (effects (font (size 1 1) (thickness 0.15)))
     )
@@
     (fp_line (start -1 0.625) (end -1 -0.625) (layer "F.Fab") (width 0.1))
     (fp_line (start 1 -0.625) (end 1 0.625) (layer "F.Fab") (width 0.1))
-    (pad "1" smd roundrect (at -0.9125 0) (size 1.025 1.4) (layers "F.Cu" "F.Paste" "F.Mask") (roundrect_rratio 0.243902)
+    (pad "1" smd roundrect (at -0.9125 0) (size 1.025 1.4) (layers "F.Cu" "F.Paste" "F.Mask") (roundrect_rratio 0.243902439)
       (net 1 "GND") (pintype "passive"))
-    (pad "2" smd roundrect (at 0.9125 0) (size 1.025 1.4) (layers "F.Cu" "F.Paste" "F.Mask") (roundrect_rratio 0.243902)
+    (pad "2" smd roundrect (at 0.9125 0) (size 1.025 1.4) (layers "F.Cu" "F.Paste" "F.Mask") (roundrect_rratio 0.243902439)
       (net 19 "Net-(D2-Pad1)") (pintype "passive"))
     (model "${KICAD6_3DMODEL_DIR}/Resistor_SMD.3dshapes/R_0805_2012Metric.wrl"
@@
     (property "Sheetname" "")
     (attr smd)
-    (fp_text reference "Rsense1" (at -0.003 -1.905) (layer "F.SilkS")
+    (fp_text reference "Rsense1" (at -1.4 -1.905) (layer "F.SilkS")
       (effects (font (size 1 1) (thickness 0.15)))
     )
@@
     (fp_line (start -1 0.625) (end -1 -0.625) (layer "F.Fab") (width 0.1))
     (fp_line (start 1 -0.625) (end 1 0.625) (layer "F.Fab") (width 0.1))
-    (pad "1" smd roundrect (at -0.9125 0) (size 1.025 1.4) (layers "F.Cu" "F.Paste" "F.Mask") (roundrect_rratio 0.243902)
+    (pad "1" smd roundrect (at -0.9125 0) (size 1.025 1.4) (layers "F.Cu" "F.Paste" "F.Mask") (roundrect_rratio 0.243902439)
       (net 46 "Net-(Ruv1-Pad1)") (pintype "passive"))
-    (pad "2" smd roundrect (at 0.9125 0) (size 1.025 1.4) (layers "F.Cu" "F.Paste" "F.Mask") (roundrect_rratio 0.243902)
+    (pad "2" smd roundrect (at 0.9125 0) (size 1.025 1.4) (layers "F.Cu" "F.Paste" "F.Mask") (roundrect_rratio 0.243902439)
       (net 1 "GND") (pintype "passive"))
     (model "${KICAD6_3DMODEL_DIR}/Resistor_SMD.3dshapes/R_0805_2012Metric.wrl"
@@
     (fp_line (start 1 -0.625) (end 1 0.625) (layer "F.Fab") (width 0.1))
     (fp_line (start -1 -0.625) (end 1 -0.625) (layer "F.Fab") (width 0.1))
-    (pad "1" smd roundrect (at -0.9125 0) (size 1.025 1.4) (layers "F.Cu" "F.Paste" "F.Mask") (roundrect_rratio 0.243902)
+    (pad "1" smd roundrect (at -0.9125 0) (size 1.025 1.4) (layers "F.Cu" "F.Paste" "F.Mask") (roundrect_rratio 0.243902439)
       (net 51 "Vin") (pintype "passive"))
-    (pad "2" smd roundrect (at 0.9125 0) (size 1.025 1.4) (layers "F.Cu" "F.Paste" "F.Mask") (roundrect_rratio 0.243902)
+    (pad "2" smd roundrect (at 0.9125 0) (size 1.025 1.4) (layers "F.Cu" "F.Paste" "F.Mask") (roundrect_rratio 0.243902439)
       (net 46 "Net-(Ruv1-Pad1)") (pintype "passive"))
     (model "${KICAD6_3DMODEL_DIR}/Resistor_SMD.3dshapes/R_0805_2012Metric.wrl"
@@
   )
   (footprint "Capacitor_SMD:C_0805_2012Metric" (layer "F.Cu")
-    (at 111.506 99.822 180)
+    (at 111.506 99.314 180)
     (descr "Capacitor SMD 0805 (2012 Metric), square (rectangular) end terminal, IPC_7351 nominal, (Body size source: IPC-SM-782 page 76, https://www.pcb-3d.com/wordpress/wp-content/uploads/ipc-sm-782a_amendment_1_and_2.pdf, https://docs.google.com/spreadsheets/d/1BsfQQcO9C6DZCsRaXUlFlo91Tg2WpOkGARC1WS5S8t0/edit?usp=sharing), generated with kicad-footprint-generator")
     (tags "capacitor")
@@
     (property "Sheetname" "")
     (attr smd)
-    (fp_text reference "Rfbb1" (at 0 -2.032) (layer "F.SilkS")
+    (fp_text reference "Rfbb1" (at 4.0595 0) (layer "F.SilkS")
       (effects (font (size 1 1) (thickness 0.15)))
     )
@@
     (fp_line (start -1 -0.625) (end 1 -0.625) (layer "F.Fab") (width 0.1))
     (fp_line (start 1 0.625) (end -1 0.625) (layer "F.Fab") (width 0.1))
-    (pad "1" smd roundrect (at -0.9125 0) (size 1.025 1.4) (layers "F.Cu" "F.Paste" "F.Mask") (roundrect_rratio 0.243902)
+    (pad "1" smd roundrect (at -0.9125 0) (size 1.025 1.4) (layers "F.Cu" "F.Paste" "F.Mask") (roundrect_rratio 0.243902439)
       (net 13 "Net-(Ccomp1-Pad1)") (pintype "passive"))
-    (pad "2" smd roundrect (at 0.9125 0) (size 1.025 1.4) (layers "F.Cu" "F.Paste" "F.Mask") (roundrect_rratio 0.243902)
+    (pad "2" smd roundrect (at 0.9125 0) (size 1.025 1.4) (layers "F.Cu" "F.Paste" "F.Mask") (roundrect_rratio 0.243902439)
       (net 1 "GND") (pintype "passive"))
     (model "${KICAD6_3DMODEL_DIR}/Resistor_SMD.3dshapes/R_0805_2012Metric.wrl"
@@
     (fp_line (start 1.6 -0.8) (end 1.6 0.8) (layer "F.Fab") (width 0.1))
     (fp_line (start -1.6 0.8) (end -1.6 -0.8) (layer "F.Fab") (width 0.1))
-    (pad "1" smd roundrect (at -1.475 0 90) (size 1.15 1.8) (layers "F.Cu" "F.Paste" "F.Mask") (roundrect_rratio 0.217391)
+    (pad "1" smd roundrect (at -1.475 0 90) (size 1.15 1.8) (layers "F.Cu" "F.Paste" "F.Mask") (roundrect_rratio 0.2173913043)
       (net 9 "/P5V") (pintype "passive"))
-    (pad "2" smd roundrect (at 1.475 0 90) (size 1.15 1.8) (layers "F.Cu" "F.Paste" "F.Mask") (roundrect_rratio 0.217391)
+    (pad "2" smd roundrect (at 1.475 0 90) (size 1.15 1.8) (layers "F.Cu" "F.Paste" "F.Mask") (roundrect_rratio 0.2173913043)
       (net 1 "GND") (pintype "passive"))
     (model "${KICAD6_3DMODEL_DIR}/Capacitor_SMD.3dshapes/C_1206_3216Metric.wrl"
@@
   (gr_arc (start 140.546356 60.817611) (mid 142.667676 61.696291) (end 143.546356 63.817611) (layer "Edge.Cuts") (width 0.1))
   (gr_arc (start 83.566 96.266) (mid 83.26842 96.98442) (end 82.55 97.282) (layer "Edge.Cuts") (width 0.1))
-  (gr_text "order q2 & lm5116" (at 101.854 50.292) (layer "F.Cu")
-    (effects (font (size 1.5 1.5) (thickness 0.3)))
-  )
   (gr_text "JLCJLCJLCJLC" (at 141.732 101.346 90) (layer "B.SilkS")
     (effects (font (size 1.5 1.5) (thickness 0.3)))
@@
   (segment (start 109.351 92.841) (end 109.351 93.341) (width 0.3) (layer "F.Cu") (net 1))
   (segment (start 122.8 68.195) (end 122.8 72.005) (width 0.2) (layer "F.Cu") (net 1))
-  (via (at 109.22 99.06) (size 0.4) (drill 0.2) (layers "F.Cu" "B.Cu") (free) (net 1))
+  (via (at 109.22 98.806) (size 0.4) (drill 0.2) (layers "F.Cu" "B.Cu") (free) (net 1))
   (via (at 102.616 76.454) (size 0.4) (drill 0.2) (layers "F.Cu" "B.Cu") (free) (net 1))
   (via (at 109.22 95.758) (size 0.4) (drill 0.2) (layers "F.Cu" "B.Cu") (net 1))
@@
   (via (at 108.5235 93.6605) (size 0.4) (drill 0.2) (layers "F.Cu" "B.Cu") (net 1))
   (via (at 95.504 103.632) (size 0.4) (drill 0.2) (layers "F.Cu" "B.Cu") (free) (net 1))
-  (via (at 109.22 100.076) (size 0.4) (drill 0.2) (layers "F.Cu" "B.Cu") (free) (net 1))
+  (via (at 109.22 99.822) (size 0.4) (drill 0.2) (layers "F.Cu" "B.Cu") (free) (net 1))
   (segment (start 119.003 68.195) (end 117.4 68.195) (width 0.25) (layer "F.Cu") (net 2))
   (segment (start 117.4 68.195) (end 115.4575 68.195) (width 0.25) (layer "F.Cu") (net 2))
@@
     (polygon
       (pts
-        (xy 85.852 92.964)
-        (xy 91.44 92.964)
+        (xy 85.852 90.932)
+        (xy 91.44 90.932)
         (xy 91.44 98.298)
         (xy 84.836 98.298)
