File: 5116-05/LM5116-05.kicad_pcb (KiCad board)
At the start: 2 copper layers, 65 x 56 mm, 50 parts, among them J1 Input, J3 40HAT, J6 CONN_02X02, J9 CONN_01X02, Q1 DMG2305UX, Q2 DMMT5401, Q3 CSD19534Q5A, Q4 IPB027N10N3_G, U1 LM5116MHX_NOPB, U2 CAT24C32

Commit message: updating working tree
Parts:
- moved Ccomp1 0.76 mm to (117.0, 89.2)
- moved J1 0.76 mm to (99.3, 109.2)
- moved Rfbb1 0.76 mm to (118.6, 87.1)
- moved Rcomp1 0.30 mm to (115.2, 90.4)
Routing:
- net GND: vias 16 -> 20
Other:
- board text added: "100pF"
- board text added: "3.3v"
- board text added: "elongate q3 footprint"
- board text added: "rev.04 mar2023 // keyudits"
- board text removed: "rev.03 feb2023 // keyudits"
Changed lines of the file:
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@@
       (drillshape 0)
       (scaleselection 1)
-      (outputdirectory "05_gerber/")
+      (outputdirectory "05_gerber/v04_gerber/")
     )
   )
@@
     (property "Sheetname" "")
     (attr smd)
-    (fp_text reference "D2" (at -0.254 1.778) (layer "F.SilkS")
+    (fp_text reference "D2" (at 2.794 0.254) (layer "F.SilkS")
       (effects (font (size 1 1) (thickness 0.15)))
     )
@@
   )
   (footprint "TerminalBlock:TerminalBlock_bornier-2_P5.08mm" (layer "F.Cu")
-    (at 99.314 108.458 180)
+    (at 99.314 109.22 180)
     (descr "simple 2-pin terminal block, pitch 5.08mm, revamped version of bornier2")
     (tags "terminal block bornier2")
@@
     (property "Sheetname" "")
     (attr smd)
-    (fp_text reference "U1" (at 0 0) (layer "F.SilkS")
+    (fp_text reference "U1" (at 2.417 -4.572) (layer "F.SilkS")
       (effects (font (size 1.27 1.27) (thickness 0.254)))
     )
@@
   )
   (footprint "Resistor_SMD:R_0805_2012Metric" (layer "F.Cu")
-    (at 118.6225 87.884)
+    (at 118.6225 87.122)
     (descr "Resistor SMD 0805 (2012 Metric), square (rectangular) end terminal, IPC_7351 nominal, (Body size source: IPC-SM-782 page 72, https://www.pcb-3d.com/wordpress/wp-content/uploads/ipc-sm-782a_amendment_1_and_2.pdf), generated with kicad-footprint-generator")
     (tags "resistor")
@@
   )
   (footprint "Capacitor_SMD:C_0402_1005Metric" (layer "F.Cu")
-    (at 116.971 89.916 180)
+    (at 116.971 89.154 180)
     (descr "Capacitor SMD 0402 (1005 Metric), square (rectangular) end terminal, IPC_7351 nominal, (Body size source: http://www.tortai-tech.com/upload/download/2011102023233369053.pdf), generated with kicad-footprint-generator")
     (tags "capacitor")
@@
   )
   (footprint "Resistor_SMD:R_0402_1005Metric" (layer "F.Cu")
-    (at 115.17 90.701 90)
+    (at 115.17 90.401 90)
     (descr "Resistor SMD 0402 (1005 Metric), square (rectangular) end terminal, IPC_7351 nominal, (Body size source: http://www.tortai-tech.com/upload/download/2011102023233369053.pdf), generated with kicad-footprint-generator")
     (tags "resistor")
@@
     (effects (font (size 1.5 1.5) (thickness 0.3)))
   )
-  (gr_text "rev.03 feb2023 // keyudits" (at 129.54 115.57) (layer "F.SilkS")
+  (gr_text "3.3v" (at 105.664 70.358) (layer "F.SilkS")
+    (effects (font (size 0.75 0.75) (thickness 0.1)))
+  )
+  (gr_text "rev.04 mar2023 // keyudits" (at 129.54 115.57) (layer "F.SilkS")
     (effects (font (size 0.6 0.6) (thickness 0.09)))
   )
-  (gr_text "+" (at 94.234 113.284 90) (layer "F.SilkS")
+  (gr_text "+" (at 94.234 115.062 90) (layer "F.SilkS")
     (effects (font (size 1.5 1.5) (thickness 0.3)))
   )
-  (gr_text "dc input" (at 97.282 114.808) (layer "F.SilkS")
+  (gr_text "100pF" (at 127.508 96.52) (layer "F.SilkS")
+    (effects (font (size 0.75 0.75) (thickness 0.1)))
+  )
+  (gr_text "dc input" (at 106.172 115.062) (layer "F.SilkS")
     (effects (font (size 0.6 0.6) (thickness 0.09)))
   )
-  (gr_text "-" (at 99.568 113.284 180) (layer "F.SilkS")
+  (gr_text "-" (at 99.314 115.316 180) (layer "F.SilkS")
     (effects (font (size 1.5 1.5) (thickness 0.3)))
+  )
+  (gr_text "elongate q3 footprint" (at 71.374 99.06) (layer "Cmts.User")
+    (effects (font (size 0.6 0.6) (thickness 0.09)))
   )
   (gr_text "cutout area (plated)" (at 123.444 105.156 90) (layer "F.Fab")
@@
   (via (at 108.458 92.964) (size 0.4) (drill 0.2) (layers "F.Cu" "B.Cu") (net 1))
   (via (at 95.25 77.724) (size 0.4) (drill 0.2) (layers "F.Cu" "B.Cu") (free) (net 1))
+  (via (at 119.126 85.598) (size 0.4) (drill 0.2) (layers "F.Cu" "B.Cu") (free) (net 1))
+  (via (at 119.634 88.646) (size 0.4) (drill 0.2) (layers "F.Cu" "B.Cu") (free) (net 1))
   (via (at 96.012 77.724) (size 0.4) (drill 0.2) (layers "F.Cu" "B.Cu") (free) (net 1))
+  (via (at 119.126 88.646) (size 0.4) (drill 0.2) (layers "F.Cu" "B.Cu") (free) (net 1))
   (via (at 109.351 93.726) (size 0.4) (drill 0.2) (layers "F.Cu" "B.Cu") (net 1))
   (via (at 108.5235 95.758) (size 0.4) (drill 0.2) (layers "F.Cu" "B.Cu") (net 1))
@@
   (via (at 108.5235 93.6605) (size 0.4) (drill 0.2) (layers "F.Cu" "B.Cu") (net 1))
   (via (at 95.504 103.632) (size 0.4) (drill 0.2) (layers "F.Cu" "B.Cu") (free) (net 1))
+  (via (at 119.634 85.598) (size 0.4) (drill 0.2) (layers "F.Cu" "B.Cu") (free) (net 1))
   (via (at 109.22 99.822) (size 0.4) (drill 0.2) (layers "F.Cu" "B.Cu") (free) (net 1))
   (segment (start 119.003 68.195) (end 117.4 68.195) (width 0.25) (layer "F.Cu") (net 2))
@@
   (segment (start 103.632 97.028) (end 103.632 95.758) (width 0.3) (layer "F.Cu") (net 11))
   (segment (start 103.987 96.113) (end 103.632 95.758) (width 0.3) (layer "F.Cu") (net 11))
-  (segment (start 115.17 90.216) (end 115.47 89.916) (width 0.4) (layer "F.Cu") (net 12))
-  (segment (start 115.47 89.916) (end 116.486 89.916) (width 0.4) (layer "F.Cu") (net 12))
-  (segment (start 114.893 87.122) (end 116.948 87.122) (width 0.4) (layer "F.Cu") (net 13))
+  (segment (start 115.932 89.154) (end 116.486 89.154) (width 0.4) (layer "F.Cu") (net 12))
+  (segment (start 115.17 89.916) (end 115.932 89.154) (width 0.4) (layer "F.Cu") (net 12))
+  (segment (start 114.893 87.122) (end 117.71 87.122) (width 0.4) (layer "F.Cu") (net 13))
   (segment (start 117.41 91.818282) (end 116.814282 92.414) (width 0.4) (layer "F.Cu") (net 13))
   (segment (start 117.71 87.884) (end 117.71 89.662) (width 0.4) (layer "F.Cu") (net 13))
@@
   (segment (start 117.41 89.962) (end 117.456 89.916) (width 0.4) (layer "F.Cu") (net 13))
   (segment (start 117.41 91.694) (end 117.41 91.818282) (width 0.4) (layer "F.Cu") (net 13))
-  (segment (start 116.948 87.122) (end 117.71 87.884) (width 0.4) (layer "F.Cu") (net 13))
   (segment (start 114.799 92.414) (end 114.35 92.863) (width 0.4) (layer "F.Cu") (net 13))
   (segment (start 116.814282 92.414) (end 114.799 92.414) (width 0.4) (layer "F.Cu") (net 13))
